Commit message: fix lidar position in urdf

File: rosbot_description/urdf/rosbot.xacro (robot description, xacro)
@@ -26,10 +26,10 @@
       </geometry>
     </collision>
-    <visual name='base_link_visual'>
+    <!-- <visual name='base_link_visual'>
       <origin xyz="0 0 -0.02" rpy=" 1.5707 0 1.5707"/>
       <geometry>
         <mesh filename="package://rosbot_description/meshes/box.dae" scale="0.001 0.001 0.001" />
       </geometry>
-    </visual>
+    </visual> -->
   </link>
   <joint name="top_joint" type="fixed">
@@ -246,5 +246,5 @@
   </transmission>
   <!-- Orbbec Astra RGBD Camera -->
-  <joint name="astra_joint" type="fixed">
+  <!-- <joint name="astra_joint" type="fixed">
     <axis xyz="0 0 0" />
     <origin xyz="-0.03 0 0.18" rpy="0 0 0"/>
@@ -284,15 +284,15 @@
   </joint>
   <link name="camera_depth_frame">
-  </link>
+  </link> -->
+  <!-- rplidar Laser -->
   <joint name="rplidar_joint" type="fixed">
     <axis xyz="0 1 0" />
-    <origin xyz="0.02 0 0" rpy="0 0 3.14"/>
+    <origin xyz="0.02 0 0.07" rpy="0 0 3.14"/>
     <parent link="base_link"/>
     <child link="laser"/>
   </joint>
-  <!-- rplidar Laser -->
   <link name="laser">
     <collision>
-      <origin xyz="0 0 0.058" rpy="1.5707 0 4.71"/>
+      <origin xyz="0 0 -.02" rpy="1.5707 0 4.71"/>
       <geometry>
         <mesh filename="package://rosbot_description/meshes/rplidar.dae" scale="0.001 0.001 0.001" />
@@ -300,5 +300,5 @@
     </collision>
     <visual>
-      <origin xyz="0 0 0.058" rpy="1.5707 0 4.71"/>
+      <origin xyz="0 0 -.02" rpy="1.5707 0 4.71"/>
       <geometry>
         <mesh filename="package://rosbot_description/meshes/rplidar.dae" scale="0.001 0.001 0.001" />
@@ -307,5 +307,5 @@
     <inertial>
       <mass value="1e-5" />
-      <origin xyz="0 0 0.058" rpy="1.5707 0 4.71"/>
+      <origin xyz="0 0 -.02" rpy="1.5707 0 4.71"/>
       <inertia ixx="0" ixy="0" ixz="0" iyy="0" iyz="0" izz="0" />
     </inertial>

Commit message: use gpu for lidar simulation

File: rosbot_description/urdf/rosbot.xacro (robot description, xacro)
@@ -26,10 +26,10 @@
       </geometry>
     </collision>
-    <!-- <visual name='base_link_visual'>
+    <visual name='base_link_visual'>
       <origin xyz="0 0 -0.02" rpy=" 1.5707 0 1.5707"/>
       <geometry>
         <mesh filename="package://rosbot_description/meshes/box.dae" scale="0.001 0.001 0.001" />
       </geometry>
-    </visual> -->
+    </visual>
   </link>
   <joint name="top_joint" type="fixed">
@@ -246,5 +246,5 @@
   </transmission>
   <!-- Orbbec Astra RGBD Camera -->
-  <!-- <joint name="astra_joint" type="fixed">
+  <joint name="astra_joint" type="fixed">
     <axis xyz="0 0 0" />
     <origin xyz="-0.03 0 0.18" rpy="0 0 0"/>
@@ -284,9 +284,9 @@
   </joint>
   <link name="camera_depth_frame">
-  </link> -->
+  </link>
   <!-- rplidar Laser -->
   <joint name="rplidar_joint" type="fixed">
     <axis xyz="0 1 0" />
-    <origin xyz="0.02 0 0.07" rpy="0 0 3.14"/>
+    <origin xyz="0.02 0 0.085" rpy="0 0 3.14"/>
     <parent link="base_link"/>
     <child link="laser"/>
@@ -294,5 +294,5 @@
   <link name="laser">
     <collision>
-      <origin xyz="0 0 -.02" rpy="1.5707 0 4.71"/>
+      <origin xyz="0 0 -.03" rpy="1.5707 0 4.71"/>
       <geometry>
         <mesh filename="package://rosbot_description/meshes/rplidar.dae" scale="0.001 0.001 0.001" />
@@ -300,5 +300,5 @@
     </collision>
     <visual>
-      <origin xyz="0 0 -.02" rpy="1.5707 0 4.71"/>
+      <origin xyz="0 0 -.03" rpy="1.5707 0 4.71"/>
       <geometry>
         <mesh filename="package://rosbot_description/meshes/rplidar.dae" scale="0.001 0.001 0.001" />
@@ -307,5 +307,5 @@
     <inertial>
       <mass value="1e-5" />
-      <origin xyz="0 0 -.02" rpy="1.5707 0 4.71"/>
+      <origin xyz="0 0 -.03" rpy="1.5707 0 4.71"/>
       <inertia ixx="0" ixy="0" ixz="0" iyy="0" iyz="0" izz="0" />
     </inertial>
